File: BLE_SoilMostureSensor/SparkFun_Soil_Moisture_Sensor.sch (EAGLE design)
At the start: 30 parts, among them Q1 2N3904, U2 EFR32BG13

Commit message: updating Soil Moisture Design
Parts:
- removed J1: (no value), SparkFun-Connectors:CONN_05X20.05_IN_PTH_SILK
- added C10: 1.5pF, SparkFun-Capacitors:1.5PF-0603-50V-16.667%
- added C11: 0.1uF, SparkFun-Capacitors:0.1UF-0603-25V-(+80/-20%)
- added C12, C14: 10pF, SparkFun-Capacitors:10PF-0603-50V-5%
- added C13: 0.22uF, SparkFun-Capacitors:0.22UF-0603-25V-10%
- added E1: ANTENNA-GROUNDEDTRACE-15.2MM, SparkFun-RF:ANTENNA-GROUNDEDTRACE-15.2MM
- added FB1, FB2: L103, SparkFun-Coils:FERRITE_BEAD-0603
- added FID1, FID2: FIDUCIAL"", microbuilder:FIDUCIAL""
- added FRAME2: FRAME-LETTER, SparkFun-Aesthetics:FRAME-LETTER
- added L2, L4: 1.9NH, SparkFun-Coils:INDUCTOR-0402-3.9NH
- added R10: 10M, SparkFun-Resistors:10MOHM-0603-1/10W-5%
- added R9: 0, SparkFun-Resistors:0.22OHM-0805-1/4W-1%
- added X1: 20317, microbuilder:JTAG-CORTEXBOXPOSTS
- BT1: device SparkFun-Batteries:BATTERY-12MM_SMD -> SparkFun-Batteries:BATTERY-20MM_SMD_4LEGS_OVERPASTE
Connections:
- net N$21 renamed ION
- removed net N$2: U2.RFVDD
- removed net N$22: U2.2G4RF_IOP
- removed net N$24: U2.RFVSS
- removed net N$25: U2.PAVSS
- removed net N$27: U2.PD15
- removed net N$5: U2.PF0
- removed net N$6: U2.PF1
- removed net N$7: U2.PF2
- removed net N$8: U2.PF3
- removed net SWCH: U$2.IN1, U$2.IN2, U$2.IN3, U$2.IN4
- removed net VCC: U$2.COM1, U$2.COM3, U$2.VCC
- new net IOP: L2.1, U2.2G4RF_IOP
- new net N$23: L4.1, R9.2
- new net N$26: E1.SIGNAL, L4.2
- new net N$3: C10.2, L2.2, R9.1
- new net N$51: X1.KEY
- new net N$52: X1.GNDDETECT
- new net N$57: X1.NRESET
- new net RFVDD: C11.1, C12.1, FB1.2, U2.RFVDD
- new net SENSOR_ENABLE: R10.2, U$2.IN1, U$2.IN2, U$2.IN3, U$2.IN4, U2.PD15
- new net TCK: U2.PF0, X1.SWDCLK
- new net TDI: U2.PF3, X1.TDI
- new net TDO: U2.PF2, X1.SWO
- new net TMS: U2.PF1, X1.SWDIO
- net GND: now also C10.1, C11.2, C12.2, C13.2, C14.2, E1.GND, R10.1, U2.PAVSS, U2.RFVSS, X1.GND@1, X1.GND@2
- net PAVDD: now also C13.1, C14.1, FB2.1, FB2.2
- net VDCDC: now also FB1.1
- net VMCU: now also X1.VCC
- net V_BATT: now also U$2.COM1, U$2.COM3, U$2.VCC
Other:
- note added: "SWD PROGRAMMER"
